File: ESP32_TOOLS.kicad_pcb (KiCad board)
At the start: 2 copper layers, 11 parts, among them J1 LED, J3 OLED, SW1 UP_SW, SW2 DOWN_SW, SW3 OK_SW, SW4 LEFT_SW, SW5 RIGHT_SW

Commit message: fofo1
Parts:
- NRF24L01_Breakout1, NRF24L01_Breakout2, NRF24L01_Breakout3: moved to B.Cu
- moved S1 59.9 mm to (152.5, 67.6), turned to 90 degrees
- moved J3 43.4 mm to (163.6, 81.7)
- moved SW5 43.0 mm to (210.1, 86.5), turned to 180 degrees
- moved SW3 41.7 mm to (199.9, 86.5), turned to 180 degrees
- moved SW4 40.4 mm to (189.8, 86.5), turned to 180 degrees
- moved SW1 37.2 mm to (193.4, 71.8)
- moved SW2 36.3 mm to (193.4, 92.2)
- moved NRF24L01_Breakout1 6.96 mm to (208.3, 57.1)
- moved NRF24L01_Breakout2 3.55 mm to (184.2, 57.1)
- moved NRF24L01_Breakout3 2.81 mm to (161.0, 57.1)
Routing:
- net /MISO: track 0.00 -> 62.1 mm, vias 0 -> 4
- net /MOSI: track 0.00 -> 61.4 mm, vias 0 -> 4
- net /SCK: track 0.00 -> 57.7 mm, vias 0 -> 4
- net /SS_ALTO: track 0.00 -> 41.8 mm
- net /CE_ALTO: track 0.00 -> 33.8 mm
- net /SS_CENTRO: track 0.00 -> 27.0 mm
- net /SS_BASSO: track 0.00 -> 24.8 mm
- net /CE_BASSO: track 0.00 -> 13.3 mm
- net /CE_CENTRO: track 0.00 -> 11.1 mm

Commit message: small corrections
Parts:
- removed J1: LED, 0Planck_20250924:PinHeader_1x03_P2.54mm_Vertical
- added ?: , , F.Cu at (164.6, 57.1)
- added ?: , , F.Cu at (208.3, 59.9)
- added ?: , , F.Cu at (187.7, 57.1)
- moved SW5 6.49 mm to (206.6, 81.0), turned to -90 degrees
- moved SW3 5.88 mm to (197.8, 81.0), turned to -90 degrees
- moved SW4 5.51 mm to (189.4, 81.0), turned to -90 degrees
- moved J3 1.46 mm to (165.1, 81.7)
- moved SW2 1.30 mm to (192.3, 91.4)
- moved SW1 1.08 mm to (192.3, 71.8)
Routing:
- net +3V3: track 0.00 -> 129.4 mm, vias 0 -> 3
- net /DOWN_SW: track 0.00 -> 119.0 mm
- net /LEFT_SW: track 0.00 -> 100.7 mm
- net /RIGHT_SW: track 0.00 -> 91.0 mm
- net /UP_SW: track 0.00 -> 86.6 mm
- net /OK_SW: track 0.00 -> 82.8 mm, vias 0 -> 1
- net /SCL: track 0.00 -> 35.4 mm
- net /MOSI: track 61.4 -> 96.0 mm, vias 4 -> 1
- net /MISO: track 62.1 -> 94.2 mm
- net /SDA: track 0.00 -> 24.8 mm
- net GND: track 0.00 -> 9.91 mm
- net /SCK: track 57.7 -> 64.6 mm, vias 4 -> 1
- net /CE_ALTO: track 33.8 -> 31.5 mm, vias 0 -> 1
- net /SS_CENTRO: track 27.0 -> 24.9 mm, vias 0 -> 1
- net /SS_BASSO: track 24.8 -> 23.9 mm, vias 0 -> 1
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- added copper zone on B.Cu, net GND
Other:
- board outline added: 68 x 67 mm
- board text added: "Copiright © 2025 ToffoJr inc. All Rights are reservated."
- board text added: "GPIO26"
